File: shift_register/shift register.brd (EAGLE design)
At the start: 160 x 100 mm, 39 parts

Commit message: gerber files
Connections:
- net N$34 renamed SRCLK
- net N$35 renamed RCLK
- removed net N$33: IC1.9, IC2.14
- removed net N$36: IC1.14, J1.3
- removed net N$37: IC2.9, J2.3
- new net QH': IC1.14, IC2.9
- new net QH'2: IC1.9, J2.3
- new net SER: IC2.14, J1.3
Routing:
- net QH'2: track 0.00 -> 97.7 mm, vias 0 -> 2
- net N$33: track 66.8 -> 0.00 mm, vias 3 -> 0
- net SER: track 0.00 -> 63.5 mm, vias 0 -> 2
- net QH': track 0.00 -> 38.3 mm
- net N$37: track 34.1 -> 0.00 mm, vias 4 -> 0
- net N$36: track 26.6 -> 0.00 mm, vias 4 -> 0
- net GND: track 592.2 -> 579.7 mm
- net 5V: track 163.6 -> 153.5 mm, vias 10 -> 6
- net SRCLK: track 94.6 -> 99.4 mm, vias 8 -> 4
- net RCLK: track 85.7 -> 86.8 mm
Other:
- board size 160 x 100 mm -> 91.4 x 75.9 mm
