File: shift_register/shift register.sch (EAGLE design)
At the start: 39 parts

Commit message: gerber files
Connections:
- net N$34 renamed SRCLK
- net N$35 renamed RCLK
- removed net N$33: IC1.9, IC2.14
- removed net N$36: IC1.14, J1.3
- removed net N$37: IC2.9, J2.3
- new net QH': IC1.14, IC2.9
- new net QH'2: IC1.9, J2.3
- new net SER: IC2.14, J1.3
Other:
- note removed: "6 - GND 5 - SHIFT REGISTER 4 - LATCH 3 - DATA 2 - GND 1 - +5v"
